File: 50x50 2 Layer Example/50x50 2 Layer.kicad_sch (KiCad schematic)
At the start: 74 parts, among them J1 Conn_01x02, J2 USB_C_Receptacle_USB2.0_14P, J3 Conn_01x03, J4 Conn_01x04, Q1 MMBT3904, SW1 PWR_SELECT, SW2 ON_SW, SW3 Reset, U1 W25Q32JVSSIQ, U2 USBLC6-2SC6, U3 Voltage Regulator (MCP1755S-3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, U4 RP2354A, U5 Sensor Board, Y1 12MHz

Commit message: Added Footprints
Added footprints for the Buzzer, 3.3uH Inductor, and the SPDT Power Switches
Parts:
- BZ1: footprint (none) -> Buzzer_Beeper:MagneticBuzzer_CUI_CST-931RP-A
- L1: footprint (none) -> Inductor_SMD:L_Taiyo-Yuden_NR-40xx_HandSoldering
- SW1: footprint (none) -> Button_Switch_THT:SW_Slide_SPDT_Straight_CK_OS102011MS2Q
Changed lines of the file:
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@@
 			)
 		)
-		(property "Footprint" ""
+		(property "Footprint" "Button_Switch_THT:SW_Slide_SPDT_Straight_CK_OS102011MS2Q"
 			(at 71.12 203.2 0)
 			(hide yes)
@@
 			)
 		)
-		(property "Datasheet" ""
+		(property "Datasheet" "https://www.littelfuse.com/assetdocs/littelfuse-c-k-slide-os-series-datasheet?assetguid=f8954ac2-65ba-431f-af55-b0493370575e"
 			(at 71.12 203.2 0)
 			(hide yes)
@@
 			)
 		)
-		(property "Footprint" ""
+		(property "Footprint" "Button_Switch_THT:SW_Slide_SPDT_Straight_CK_OS102011MS2Q"
 			(at 35.56 236.22 0)
 			(hide yes)
@@
 			)
 		)
-		(property "Datasheet" ""
+		(property "Datasheet" "https://www.littelfuse.com/assetdocs/littelfuse-c-k-slide-os-series-datasheet?assetguid=f8954ac2-65ba-431f-af55-b0493370575e"
 			(at 35.56 236.22 0)
 			(hide yes)
@@
 			)
 		)
-		(property "Footprint" ""
+		(property "Footprint" "Inductor_SMD:L_Taiyo-Yuden_NR-40xx_HandSoldering"
 			(at 233.68 160.02 0)
 			(hide yes)
@@
 			)
 		)
-		(property "Datasheet" ""
+		(property "Datasheet" "https://mm.digikey.com/Volume0/opasdata/d220001/medias/docus/610/NRS4018T3R3MDGJ_SS.pdf"
 			(at 233.68 160.02 0)
 			(hide yes)
@@
 			)
 		)
-		(property "Footprint" ""
+		(property "Footprint" "Buzzer_Beeper:MagneticBuzzer_CUI_CST-931RP-A"
 			(at 276.225 85.09 90)
 			(hide yes)
@@
 			)
 		)
-		(property "Datasheet" ""
+		(property "Datasheet" "https://www.sameskydevices.com/product/resource/cst-931ap.pdf"
 			(at 276.225 85.09 90)
 			(hide yes)
