File: 50x50 2 Layer Example/_autosave-50x50 2 Layer.kicad_sch (KiCad schematic)
At the start: 73 parts, among them J1 Conn_01x02, J2 USB_C_Receptacle_USB2.0_14P, J3 Conn_01x03, J4 Conn_01x04, Q1 MMBT3904, SW1 PWR_SELECT, SW3 Reset, SW4 ON_SW, U1 W25Q32JVSSIQ, U2 USBLC6-2SC6, U3 Voltage Regulator (MCP1755S-3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, U4 RP2354A, U5 Sensor Board, Y1 12MHz

Commit message: Updated Inductor
Other:
- moved on the sheet: J4
Changed lines of the file:
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@@
 	(wire
 		(pts
-			(xy 363.22 154.94) (xy 373.38 154.94)
+			(xy 364.49 156.21) (xy 374.65 156.21)
 		)
 		(stroke
@@
 	(wire
 		(pts
-			(xy 394.97 189.23) (xy 389.89 189.23)
+			(xy 394.97 191.77) (xy 389.89 191.77)
 		)
 		(stroke
@@
 	(wire
 		(pts
-			(xy 363.22 157.48) (xy 373.38 157.48)
+			(xy 364.49 158.75) (xy 374.65 158.75)
 		)
 		(stroke
@@
 	(wire
 		(pts
-			(xy 361.95 189.23) (xy 372.11 189.23)
+			(xy 358.14 191.77) (xy 368.3 191.77)
 		)
 		(stroke
@@
 	(wire
 		(pts
+			(xy 368.3 184.15) (xy 358.14 184.15)
+		)
+		(stroke
+			(width 0)
+			(type default)
+		)
+	)
+	(wire
+		(pts
 			(xy 43.18 241.3) (xy 43.18 238.76)
 		)
@@
 	(wire
 		(pts
-			(xy 373.38 165.1) (xy 373.38 162.56)
+			(xy 374.65 166.37) (xy 374.65 163.83)
 		)
 		(stroke
@@
 	(wire
 		(pts
-			(xy 361.95 184.15) (xy 372.11 184.15)
-		)
-		(stroke
-			(width 0)
-			(type default)
-		)
-	)
-	(wire
-		(pts
 			(xy 219.71 57.15) (xy 219.71 58.42)
 		)
@@
 	(wire
 		(pts
-			(xy 355.6 186.69) (xy 372.11 186.69)
+			(xy 355.6 187.96) (xy 368.3 187.96)
 		)
 		(stroke
@@
 	(wire
 		(pts
-			(xy 356.87 160.02) (xy 373.38 160.02)
+			(xy 358.14 161.29) (xy 374.65 161.29)
 		)
 		(stroke
@@
 		)
 	)
-	(label "I2C1_SCL"
-		(at 361.95 184.15 0)
-		(effects
-			(font
-				(size 1.27 1.27)
-			)
-			(justify left bottom)
-		)
-	)
 	(label "USB_D+"
 		(at 243.84 181.61 0)
@@
 	)
 	(label "I2C1_SDA"
-		(at 361.95 189.23 0)
+		(at 358.14 191.77 0)
 		(effects
 			(font
@@
 		)
 	)
+	(label "I2C1_SCL"
+		(at 358.14 184.15 0)
+		(effects
+			(font
+				(size 1.27 1.27)
+			)
+			(justify left bottom)
+		)
+	)
 	(label "SPI1_SCK"
 		(at 58.42 124.46 0)
@@
 	)
 	(label "I2C0_SCL"
-		(at 363.22 157.48 0)
+		(at 364.49 158.75 0)
 		(effects
 			(font
@@
 	)
 	(label "I2C0_SDA"
-		(at 363.22 154.94 0)
+		(at 364.49 156.21 0)
 		(effects
 			(font
@@
 	(global_label "INT_1"
 		(shape output)
-		(at 355.6 186.69 180)
+		(at 355.6 187.96 180)
 		(fields_autoplaced yes)
 		(effects
@@
 		)
 		(property "Intersheetrefs" "${INTERSHEET_REFS}"
-			(at 347.5348 186.69 0)
+			(at 347.5348 187.96 0)
 			(hide yes)
 			(show_name no)
@@
 	(symbol
 		(lib_id "Connector_Generic:Conn_01x04")
-		(at 378.46 160.02 0)
+		(at 379.73 161.29 0)
 		(mirror x)
 		(unit 1)
@@
 		(dnp no)
 		(property "Reference" "J4"
-			(at 381 160.0201 0)
+			(at 382.27 161.2901 0)
 			(show_name no)
 			(do_not_autoplace no)
@@
 		)
 		(property "Value" "Conn_01x04"
-			(at 381 157.4801 0)
+			(at 382.27 158.7501 0)
 			(show_name no)
 			(do_not_autoplace no)
@@
 		)
 		(property "Footprint" "Connector_PinSocket_2.54mm:PinSocket_1x04_P2.54mm_Vertical"
-			(at 378.46 160.02 0)
+			(at 379.73 161.29 0)
 			(hide yes)
 			(show_name no)
@@
 		)
 		(property "Datasheet" "https://www.lcsc.com/datasheet/lcsc_datasheet_2207291800_ZHOURI-2-54-1-4_C5116483.pdf"
-			(at 378.46 160.02 0)
+			(at 379.73 161.29 0)
 			(hide yes)
 			(show_name no)
@@
 		)
 		(property "Description" "Generic connector, single row, 01x04, script generated (kicad-library-utils/schlib/autogen/connector/)"
-			(at 378.46 160.02 0)
+			(at 379.73 161.29 0)
 			(hide yes)
 			(show_name no)
@@
 		)
 		(property "LCSC Part Number" "C5116483"
-			(at 378.46 160.02 0)
+			(at 379.73 161.29 0)
 			(hide yes)
 			(show_name no)
@@
 		)
 		(property "MPN" "2.54-1*4"
-			(at 378.46 160.02 0)
+			(at 379.73 161.29 0)
 			(hide yes)
 			(show_name no)
@@
 	(symbol
 		(lib_id "power:GND")
-		(at 373.38 165.1 0)
+		(at 374.65 166.37 0)
 		(unit 1)
 		(body_style 1)
@@
 		(fields_autoplaced yes)
 		(property "Reference" "#PWR045"
-			(at 373.38 171.45 0)
+			(at 374.65 172.72 0)
 			(hide yes)
 			(show_name no)
@@
 		)
 		(property "Value" "GND"
-			(at 373.38 170.18 0)
+			(at 374.65 171.45 0)
 			(show_name no)
 			(do_not_autoplace no)
@@
 		)
 		(property "Footprint" ""
-			(at 373.38 165.1 0)
+			(at 374.65 166.37 0)
 			(hide yes)
 			(show_name no)
@@
 		)
 		(property "Datasheet" ""
-			(at 373.38 165.1 0)
+			(at 374.65 166.37 0)
 			(hide yes)
 			(show_name no)
@@
 		)
 		(property "Description" "Power symbol creates a global label with name \"GND\" , ground"
-			(at 373.38 165.1 0)
+			(at 374.65 166.37 0)
 			(hide yes)
 			(show_name no)
@@
 	(symbol
 		(lib_id "power:GND")
-		(at 394.97 189.23 0)
+		(at 394.97 191.77 0)
 		(unit 1)
 		(body_style 1)
@@
 		(fields_autoplaced yes)
 		(property "Reference" "#PWR048"
-			(at 394.97 195.58 0)
+			(at 394.97 198.12 0)
 			(hide yes)
 			(show_name no)
@@
 		)
 		(property "Value" "GND"
-			(at 394.97 194.31 0)
+			(at 394.97 196.85 0)
 			(show_name no)
 			(do_not_autoplace no)
@@
 		)
 		(property "Footprint" ""
-			(at 394.97 189.23 0)
+			(at 394.97 191.77 0)
 			(hide yes)
 			(show_name no)
@@
 		)
 		(property "Datasheet" ""
-			(at 394.97 189.23 0)
+			(at 394.97 191.77 0)
 			(hide yes)
 			(show_name no)
@@
 		)
 		(property "Description" "Power symbol creates a global label with name \"GND\" , ground"
-			(at 394.97 189.23 0)
+			(at 394.97 191.77 0)
 			(hide yes)
 			(show_name no)
@@
 	(symbol
 		(lib_id "Sense:Sense_Calistated")
-		(at 381 191.77 0)
+		(at 381 195.58 0)
 		(unit 1)
 		(body_style 1)
@@
 		(fields_autoplaced yes)
 		(property "Reference" "U5"
-			(at 381 179.07 0)
+			(at 379.476 178.562 0)
 			(show_name no)
 			(do_not_autoplace no)
@@
 		)
 		(property "Value" "Sensor Board"
-			(at 381 181.61 0)
+			(at 379.222 180.34 0)
 			(show_name no)
 			(do_not_autoplace no)
@@
 		)
 		(property "Footprint" "Footprints:UCA_Sense"
-			(at 381 191.77 0)
+			(at 381 195.58 0)
 			(hide yes)
 			(show_name no)
@@
 		)
 		(property "Datasheet" ""
-			(at 381 191.77 0)
+			(at 381 195.58 0)
 			(hide yes)
 			(show_name no)
@@
 		)
 		(property "Description" ""
-			(at 381 191.77 0)
+			(at 381 195.58 0)
 			(hide yes)
 			(show_name no)
@@
 		)
 		(property "LCSC Part Number" ""
-			(at 381 191.77 0)
+			(at 381 195.58 0)
 			(hide yes)
 			(show_name no)
@@
 	(symbol
 		(lib_id "power:+3V3")
-		(at 356.87 160.02 0)
+		(at 358.14 161.29 0)
 		(unit 1)
 		(body_style 1)
@@
 		(fields_autoplaced yes)
 		(property "Reference" "#PWR042"
-			(at 356.87 163.83 0)
+			(at 358.14 165.1 0)
 			(hide yes)
 			(show_name no)
@@
 		)
 		(property "Value" "+3V3"
-			(at 356.87 154.94 0)
+			(at 358.14 156.21 0)
 			(show_name no)
 			(do_not_autoplace no)
@@
 		)
 		(property "Footprint" ""
-			(at 356.87 160.02 0)
+			(at 358.14 161.29 0)
 			(hide yes)
 			(show_name no)
@@
 		)
 		(property "Datasheet" ""
-			(at 356.87 160.02 0)
+			(at 358.14 161.29 0)
 			(hide yes)
 			(show_name no)
@@
 		)
 		(property "Description" "Power symbol creates a global label with name \"+3V3\""
-			(at 356.87 160.02 0)
+			(at 358.14 161.29 0)
 			(hide yes)
 			(show_name no)

Commit message: Fixed RP2354A Schematic Added LCSC Part Numbers Added Datasheets
Parts:
- removed BZ2: Buzzer, Buzzer_Beeper:Buzzer_Murata_PKMCS0909E, symbol Device:Buzzer
- removed L1: 3.3u, Footprints:IND-SMD_L2.0-W1.6_AOTA-B201610S3R3-101-T, symbol Device:L_Small
- removed Q1: MMBT3904, Package_TO_SOT_SMD:SOT-23, symbol Transistor_BJT:MMBT3904
- removed R16: 1k, Capacitor_SMD:C_0603_1608Metric_Pad1.08x0.95mm_HandSolder, symbol Device:R
- removed U4: RP2354A, Package_DFN_QFN:QFN-60-1EP_7x7mm_P0.4mm_EP3.4x3.4mm, symbol MCU_RaspberryPi:RP2354A
- added BZ3: Buzzer, Buzzer_Beeper:Buzzer_Murata_PKMCS0909E, symbol Device:Buzzer
- added C21, C22, C23: 100n, Capacitor_SMD:C_0603_1608Metric_Pad1.08x0.95mm_HandSolder, symbol Device:C
- added C24: 10u, Capacitor_SMD:C_0805_2012Metric, symbol Device:C
- added L1: 3.3u, Footprints:IND-SMD_L2.0-W1.6_AOTA-B201610S3R3-101-T, symbol Device:L
- added Q2: MMBT3904, Package_TO_SOT_SMD:SOT-23, symbol Transistor_BJT:MMBT3904
- added R26, R27: 1k, Resistor_SMD:R_0603_1608Metric_Pad0.98x0.95mm_HandSolder, symbol Device:R
- added SW2: SW_Push, Button_Switch_SMD:SW_SPST_TS-1088-xR020, symbol Switch:SW_Push
- added U4: RP2354_60QFN, Package_DFN_QFN:QFN-60-1EP_7x7mm_P0.4mm_EP3.4x3.4mm_ThermalVias, symbol MCU_RaspberryPi_RP2350:RP2350_60QFN
- C13: value 4.7u -> 100n
- C14, C15: value 100n -> 4.7u; LCSC Part Number C28233 -> (none); MPN CL21B104KCFNNNE -> (none)
- C16, C17, C18, C19: LCSC Part Number C28233 -> (none); MPN CL21B104KCFNNNE -> (none)
- C20: value 10u -> 100n; footprint Capacitor_SMD:C_0805_2012Metric_Pad1.18x1.45mm_HandSolder -> Capacitor_SMD:C_0603_1608Metric_Pad1.08x0.95mm_HandSolder; LCSC Part Number C28323 -> (none); MPN CL21B105KBFNNNE -> (none)
- C3, C6: footprint Capacitor_SMD:C_0603_1608Metric_Pad1.08x0.95mm_HandSolder -> Capacitor_SMD:C_0805_2012Metric
- D1: value Blue LED -> Yellow LED; footprint LED_SMD:LED_0805_2012Metric_Pad1.15x1.40mm_HandSolder -> LED_SMD:LED_0805_2012Metric
- D10: value LED -> Green LED; footprint LED_SMD:LED_0402_1005Metric_Pad0.77x0.64mm_HandSolder -> LED_SMD:LED_0805_2012Metric
- D4, D5: footprint LED_SMD:LED_0805_2012Metric_Pad1.15x1.40mm_HandSolder -> LED_SMD:LED_0805_2012Metric
- D8: value LED -> Red LED; footprint LED_SMD:LED_0402_1005Metric_Pad0.77x0.64mm_HandSolder -> LED_SMD:LED_0805_2012Metric
- D9: value LED -> Yellow LED; footprint LED_SMD:LED_0402_1005Metric_Pad0.77x0.64mm_HandSolder -> LED_SMD:LED_0805_2012Metric
- R10: footprint Capacitor_SMD:C_0603_1608Metric_Pad1.08x0.95mm_HandSolder -> Resistor_SMD:R_0603_1608Metric_Pad0.98x0.95mm_HandSolder; LCSC Part Number C17414 -> (none); MPN RC0805FR-074K7L -> (none)
- R11: value 360 -> 390
- R12, R9: footprint Capacitor_SMD:C_0603_1608Metric_Pad1.08x0.95mm_HandSolder -> Resistor_SMD:R_0603_1608Metric_Pad0.98x0.95mm_HandSolder
- R13: value 27 -> 1k; footprint Capacitor_SMD:C_0603_1608Metric_Pad1.08x0.95mm_HandSolder -> Resistor_SMD:R_0603_1608Metric_Pad0.98x0.95mm_HandSolder; LCSC Part Number C17588 -> (none); MPN 0805W8F274JT5E -> (none)
- R14: footprint Capacitor_SMD:C_0603_1608Metric_Pad1.08x0.95mm_HandSolder -> Resistor_SMD:R_0603_1608Metric_Pad0.98x0.95mm_HandSolder; LCSC Part Number C17588 -> (none); MPN 0805W8F274JT5E -> (none)
- R15: value 1k -> 27; footprint Capacitor_SMD:C_0603_1608Metric_Pad1.08x0.95mm_HandSolder -> Resistor_SMD:R_0603_1608Metric_Pad0.98x0.95mm_HandSolder; MPN RC0805FR-074K7L -> (none)
- R21, R22, R23: value 80 -> 100
- R3, R6, R7, R8: footprint Resistor_SMD:R_0603_1608Metric -> Resistor_SMD:R_0603_1608Metric_Pad0.98x0.95mm_HandSolder
- SW3: value Reset -> SW_Push; footprint Button_Switch_SMD:SW_SPST_PTS645 -> Button_Switch_SMD:SW_SPST_TS-1088-xR020; LCSC Part Number C2837531 -> (none); MPN KH-6X6X5H-STM -> (none)
Connections:
- net +1V1: now also C12.1, C13.1, C15.1, C16.1, L1.1, U4.23 (DVDD), U4.39 (DVDD), U4.50 (VREG_FB), U4.6 (DVDD); no longer C12.2
- net +3V3: now also C11.1, C20.1, BZ3.1 (+), C21.1, C22.1, C23.1, C24.1, R27.1, U4.1 (IOVDD), U4.11 (IOVDD), U4.20 (IOVDD), U4.30 (IOVDD), U4.38 (IOVDD), U4.44 (ADC_AVDD), U4.45 (IOVDD), U4.49 (VREG_VIN), U4.53 (USB_OTP_VDD), U4.54 (QSPI_IOVDD); no longer C11.2, C14.1, C15.1, C16.1, C20.2
- net ADC_0: now also U4.40 (GPIO26_ADC0)
- net ADC_1: now also U4.41 (GPIO27_ADC1)
- net ADC_2: now also U4.42 (GPIO28_ADC2)
- net ADC_3: now also U4.43 (GPIO29_ADC3)
- net BUZZER: now also R26.2, U4.4 (GPIO2); no longer R15.2
- net CLK_GPIN0: now also U4.32 (GPIO20)
- net CLK_GPOUT0: now also U4.33 (GPIO21)
- net D+: no longer R14.1
- net D-: no longer R13.1
- net GND: now also C11.2, C12.2, C13.2, C20.2, C21.2, C22.2, C23.2, C24.2, Q2.2 (E), SW2.1, U4.47 (VREG_PGND), U4.61 (GND); no longer C11.1, C12.1, C13.1, C20.1
- net GPIO_3: now also U4.5 (GPIO3)
- net GPIO_4: now also U4.7 (GPIO4)
- net GPIO_5: now also U4.8 (GPIO5)
- net GPIO_6: now also U4.9 (GPIO6)
- net GPIO_7: now also U4.10 (GPIO7)
- net I2C0_SCL: now also U4.37 (GPIO25)
- net I2C0_SDA: now also U4.36 (GPIO24)
- net I2C1_SCL: now also U4.35 (GPIO23)
- net I2C1_SDA: now also U4.34 (GPIO22)
- net INT_1: now also U4.12 (GPIO8)
- net LED_GREEN: now also U4.15 (GPIO11)
- net LED_RED: now also U4.13 (GPIO9)
- net LED_RGB: now also U4.3 (GPIO1)
- net LED_YELLOW: now also U4.14 (GPIO10)
- net RUN: now also U4.26 (RUN)
- net SPI0_CSn: now also U4.28 (GPIO17)
- net SPI0_MISO: now also U4.27 (GPIO16)
- net SPI0_MOSI: now also U4.31 (GPIO19)
- net SPI0_SCK: now also U4.29 (GPIO18)
- net SPI1_CSn: now also U4.17 (GPIO13)
- net SPI1_MISO: now also U4.16 (GPIO12)
- net SPI1_MOSI: now also U4.19 (GPIO15)
- net SPI1_SCK: now also U4.18 (GPIO14)
- net SWCLK: now also U4.24 (SWCLK)
- net SWD: now also U4.25 (SWD)
- net USB_D+: now also R14.1; no longer R14.2
- net USB_D-: now also R15.1; no longer R13.2
- net USB_DET: now also U4.2 (GPIO0)
- net XIN: now also U4.21 (XIN)
- net XOUT: now also U4.22 (XOUT)
- net VREG_AVDD: now reaches R12.2
- net VREG_AVDD: now also C14.1, U4.46 (VREG_AVDD); no longer C13.2
- new net: BZ3.2 (-), Q2.3 (C), R27.2
- new net: R15.2, U4.51 (USB_DM)
- new net: R14.2, U4.52 (USB_DP)
- new net: Q2.1 (B), R26.1
- new net QSPI_SS: R13.1, U4.60 (QSPI_SS)
- new net VREG_LX: L1.2, U4.48 (VREG_LX)
- new net ~{USB_BOOT}: R13.2, SW2.2
- no-connect marks 10 -> 9
Other:
- note added: "Make sure R7 and R8 are close to RP2350"
- note added: "Raspberry Pi Microcontroller RP2354A"
- note removed: "Bypass and decoupling capacitors"
- note removed: "RP2354A"
- note removed: "Reset Button"
- moved on the sheet: C1, C10, C2, C3, C4, C5, C6, C7, C8, C9, D1, D2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
